Commit message: Changed "lens" to "lense"

File: src/my_r2d2/urdf/r2d2.urdf.xacro (robot description, xacro)
@@ -215,5 +215,5 @@
     <origin xyz="${.707*width+0.04} 0 ${.707*width}"/>
   </joint>
-  <link name="lens">
+  <link name="lense">
     <visual>
       <geometry>
@@ -231,7 +231,7 @@
     <xacro:default_inertial mass="0.5"/>
   </link>
-  <joint name="tolens" type="fixed">
+  <joint name="tolense" type="fixed">
     <parent link="box"/>
-    <child link="lens"/>
+    <child link="lense"/>
     <origin xyz="-${boxlen/2} 0 0"/>
   </joint>

Commit message: Exercise 3: robot control

File: src/my_r2d2/urdf/r2d2.urdf.xacro (robot description, xacro)
@@ -236,3 +236,10 @@
     <origin xyz="-${boxlen/2} 0 0"/>
   </joint>
+  <link name="base_footprint">
+  </link>
+  <joint name="footprint_to_base" type="fixed">
+    <parent link="base_footprint"/>
+    <child link="base_link"/>
+    <origin xyz="0 0 0.47"/>
+  </joint>
 </robot>

Commit message: Exercise 4: completed

File: src/my_r2d2/urdf/r2d2.urdf.xacro (robot description, xacro)
@@ -236,4 +236,11 @@
     <origin xyz="-${boxlen/2} 0 0"/>
   </joint>
+  <link name="eye">
+  </link>
+  <joint name="toeye" type="fixed">
+    <parent link="lense"/>
+    <child link="eye"/>
+    <origin rpy="-${pi/2} 0 -${pi/2}" xyz="0 0 0"/>
+  </joint>
   <link name="base_footprint">
   </link>
